File: v1.0-Beta-WiFi-Nugget.kicad_pcb (KiCad board)
At the start: 2 copper layers, 36 x 50 mm, 53 parts, among them J1 Micro USB, J2 JST PH 2.0, J3 JST_SH_SM03B-SRSS-TB_1x03-1MP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, Q1 UMH3N, Q2 DMG3415, SW1 SPDT, SW2 UP, SW3 Reset, SW4 DOWN, SW5 LEFT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

Commit message: v1.0 gerber + bom files
Parts:
- added Ref**: Val**, Deluxe-Nugg-Board-Art, F.Cu at (0.00, 0.00)
- moved R11 47.3 mm to (-12.2, 4.32)
- moved C10 47.3 mm to (-9.83, 6.99)
- moved Q2 47.3 mm to (-9.42, 4.27)
- moved R6 47.3 mm to (-12.1, 11.0)
- moved J2 39.1 mm to (-12.5, 14.4)
- moved C2 33.9 mm to (7.96, -6.69)
- moved C3 33.9 mm to (3.38, -6.65)
- moved R1 33.9 mm to (9.53, -6.75)
- moved R16 33.9 mm to (0.41, -6.59)
- moved R17 33.9 mm to (1.89, -6.62)
- moved C13 33.9 mm to (4.91, -6.69)
- moved D1 33.9 mm to (11.1, -6.74)
- moved Q1 33.9 mm to (-1.80, -6.49)
- moved R15 33.9 mm to (6.43, -6.69)
- moved R9 33.9 mm to (12.7, -6.75)
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Routing:
- net GNDREF: track 0.00 -> 113.2 mm, vias 0 -> 17
- net GPIO13: track 0.00 -> 76.9 mm, vias 0 -> 3
- net +3V3: track 0.00 -> 75.6 mm
- net GPIO14: track 0.00 -> 73.0 mm, vias 0 -> 2
- net GPIO12: track 0.00 -> 68.4 mm, vias 0 -> 3
- net VMAX: track 0.00 -> 67.7 mm, vias 0 -> 3
- net ESP_RST: track 0.00 -> 59.8 mm, vias 0 -> 2
- net A0: track 0.00 -> 49.2 mm, vias 0 -> 2
- net GPIO0: track 0.00 -> 48.4 mm, vias 0 -> 3
- net VBUS: track 0.00 -> 32.8 mm
- net SDA: track 0.00 -> 29.9 mm, vias 0 -> 2
- net TXD: track 0.00 -> 27.1 mm, vias 0 -> 2
- net SCL: track 0.00 -> 27.0 mm, vias 0 -> 2
- net Net-(R10-Pad2): track 0.00 -> 24.9 mm
- net DOUT: track 0.00 -> 23.4 mm, vias 0 -> 1
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- added copper zone on F.Cu, net (none)
- added copper zone on B.Cu, net GNDREF
- added copper zone on F.Cu, net GNDREF

Commit message: v1.0 board file update
Routing:
- net GNDREF: track 113.2 -> 0.00 mm, vias 17 -> 0
- net GPIO13: track 76.9 -> 0.00 mm, vias 3 -> 0
- net +3V3: track 75.6 -> 0.00 mm
- net GPIO14: track 73.0 -> 0.00 mm, vias 2 -> 0
- net GPIO12: track 68.4 -> 0.00 mm, vias 3 -> 0
- net VMAX: track 67.7 -> 0.00 mm, vias 3 -> 0
- net ESP_RST: track 59.8 -> 0.00 mm, vias 2 -> 0
- net A0: track 49.2 -> 0.00 mm, vias 2 -> 0
- net GPIO0: track 48.4 -> 0.00 mm, vias 3 -> 0
- net VBUS: track 32.8 -> 0.00 mm
- net SDA: track 29.9 -> 0.00 mm, vias 2 -> 0
- net TXD: track 27.1 -> 0.00 mm, vias 2 -> 0
- net SCL: track 27.0 -> 0.00 mm, vias 2 -> 0
- net Net-(R10-Pad2): track 24.9 -> 0.00 mm
- net DOUT: track 23.4 -> 0.00 mm, vias 1 -> 0
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